Commit message: performance optimization and refactoring

File: test/test_files/test_default_property_complex.xacro (robot description, xacro)
@@ -4,4 +4,5 @@
         <foo/>
         <xacro:property name="prop" value="true"/>
+        <xacro:include filename="test_default_property_complex_include.xacro"/>
     </xacro:unless>
     <!-- second foo should be ignored -->

File: test/test_files/test_default_property_complex_include.xacro (robot description, xacro)
@@ -3,5 +3,5 @@
     <xacro:unless value="${prop}">
         <foo/>
-        <xacro:property name="prop" value="true"/>
+        <xacro:property name="prop" value="false"/>
     </xacro:unless>
     <!-- second foo should be ignored -->
